File: SCHEMES/STM32F411E/Kitchen_Hall_Garage_Rooms/Kitchen_Hall_Garage_Rooms.sch (KiCad schematic (older format))
At the start: 28 parts, among them M1 Motor_Servo, M2 Motor_Servo, Q1 Q_NPN_CBE, U1 STM32F411VETx, U2 BMP280, U3 MSX_DS1307, U4 DHT11

Commit message: Schema corrections
Parts:
- removed U3: MSX_DS1307, symbol RTC_LIB2:MSX_DS1307
- removed U4: DHT11, Sensor:Aosong_DHT11_5.5x12.0_P2.54mm, symbol Sensor:DHT11
- added SW_Door: SW_DPST, symbol Switch:SW_DPST_x2
- added U2: RFM95W-868S2, symbol RF_Module:RFM95W-868S2
- added U3: DS1302, symbol Timer_RTC:DS1302
- gave numbers to parts that had none: 1
Connections:
- net LIGHT_DOWN is gone; now on net SUN_DOWN: R4.2.2, RP1.2.1
- net LIGHT_LEFT is gone; now on net SUN_LEFT: R4.3.2, RP1.3.1
- net LIGHT_RIGHT is gone; now on net SUN_RIGHT: R4.4.2, RP.1.4.1
- net LIGHT_UP is gone; now on net SUN_UP: R4.1.2, RP1.1.1
- net SERVO_BOTTOM is gone; now on net PWM_BOTTOM: M2.1 (PWM)
- net SERVO_TOP is gone; now on net PWM_TOP: M1.1 (PWM)
- net SPI_MISO is gone; now on net SPI_MISO_BMP: U2.5 (SDO)
- net SPI_MOSI is gone; now on net SPI_MOSI_BMP: U2.3 (SDI)
- net SPI_SCK is gone; now on net SPI_SCK_BMP: U2.4 (SCK)
- net +3V3: now also U2.13 (3.3V), U3.1 (VCC)
- net BUZZER: now also U1.45 (PE14)
- net CAR: now also U1.33 (PC4)
- net CM_ALARM_OFF: now also U1.44 (PE13)
- net CS_BMP: now also U1.47 (PB10)
- net GND: now also SW_Door.2 (B), U2.1 (GND), U2.10 (GND), U2.8 (GND), U3.2 (GND)
- net LIGHT_GARAGE: now also U1.43 (PE12)
- net LIGHT_HALL: now also U1.42 (PE11)
- net LIGHT_KITCHEN: now also U1.41 (PE10)
- net MOTION_GARAGE: now also U1.40 (PE9)
- net MOTION_HALL: now also U1.39 (PE8)
- net MOTION_KITCHEN: now also U1.38 (PE7)
- net SUN_UP: now reaches U1.15 (PC0)
- net SUN_DOWN: now reaches U1.16 (PC1)
- net SUN_RIGHT: now reaches U1.17 (PC2)
- net SUN_LEFT: now reaches U1.18 (PC3)
- net SPI1_SCK: now reaches U1.30 (PA5)
- net SPI1_SCK: now also U2.4 (SCK)
- net SPI1_MISO: now reaches U1.31 (PA6)
- net SPI1_MISO: now also U2.2 (MISO)
- net SPI1_MOSI: now reaches U1.32 (PA7)
- net SPI1_MOSI: now also U2.3 (MOSI)
- net CS_LORA: now reaches U1.35 (PB0)
- net CS_LORA: now also U2.5 (NSS)
- net RST: now reaches U1.36 (PB1)
- net RST: now also U2.6 (RESET)
- net DIO0: now reaches U1.37 (PB2)
- net DIO0: now also U2.14 (DIO0)
- net DOOR: now reaches U1.46 (PE15)
- net DOOR: now also SW_Door.1 (A)
- net SPI_SCK_BMP: now reaches U1.51 (PB12)
- net PWM_TOP: now reaches U1.52 (PB13)
- net PWM_BOTTOM: now reaches U1.53 (PB14)
- net SCLK_RTC: now reaches U1.63 (PC6)
- net SCLK_RTC: now also U3.3 (CLK)
- net SDA_RTC: now reaches U1.64 (PC7)
- net SDA_RTC: now also U3.4 (DAT)
- net RST_RTC: now reaches U1.65 (PC8)
- net RST_RTC: now also U3.5 (RST)
- net SPI_MISO_BMP: now reaches U1.79 (PC11)
- net SPI_MOSI_BMP: now reaches U1.80 (PC12)
Other:
- note added: "Radio Module\n"
- moved on the sheet: U2

Commit message: Final version
Connections:
- net PWM_BOTTOM: now also U1.60 (PD13); no longer U1.53 (PB14)
- net PWM_TOP: now also U1.59 (PD12); no longer U1.52 (PB13)
Other:
- moved on the sheet: BZ, D_Gar, D_Hall, D_Kit, M1, M2, Q1, R1, R2, R3, R4.1, R4.2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
